Commit message: add

File: FRA333-Assignment-lab2-template/lab2_ws/src/robot_23_description/robot/dummy_description.xacro (robot description, xacro)
@@ -64,5 +64,5 @@
       <origin rpy="0 0 0" xyz="0 0 0"/>
       <geometry>
-        <mesh filename="package://robot_23_description/meshes/link_3.STL"/>
+        <mesh filename="package://robot_23_description/meshes/gripper.STL"/>
       </geometry>
       <material name="Orange"/>
@@ -72,5 +72,5 @@
     <parent link="link_3"/>
     <child link="end_effector"/>
-    <origin rpy="1.57 0 1.57" xyz="0.35 0 0"/>
+    <origin rpy="1.57 0 1.57" xyz="0.16 0 0"/>
     <axis xyz="0 0 1"/>
   </joint>

Commit message: add

File: FRA333-Assignment-lab2-template/lab2_ws/src/robot_23_description/robot/dummy_description.xacro (robot description, xacro)
@@ -11,7 +11,12 @@
 </material>
 <!-- <link name="world"/> -->
-<link name="link_0">
+  <link name="base_link">
+  </link>
+  <joint name="joint_base" type="fixed">
+    <parent link="base_link"/>
+    <child link="link_0"/>
+  </joint>
+  <link name="link_0">
     <visual>
-      <origin rpy="0 0 0" xyz="0 0 0"/>
       <geometry>
         <!-- <mesh filename="package://fra333_lab1/meshes/link_0.stl"/> -->
@@ -30,5 +35,4 @@
   <link name="link_1">
     <visual>
-      <origin rpy="0 0 0" xyz="0 0 0"/>
       <geometry>
         <mesh filename="package://robot_23_description/meshes/link_1.STL"/>
@@ -73,5 +77,4 @@
     <child link="end_effector"/>
     <origin rpy="1.57 0 1.57" xyz="0.16 0 0"/>
-    <axis xyz="0 0 1"/>
   </joint>
   <link name="end_effector"> <!-- # แสดง -->

Commit message: add

File: FRA333-Assignment-lab2-template/lab2_ws/src/robot_23_description/robot/dummy_description.xacro (robot description, xacro)
@@ -10,15 +10,7 @@
   <color rgba="0.5 0.7 1.0 1.0"/>
 </material>
-<!-- <link name="world"/> -->
-  <link name="base_link">
-  </link>
-  <joint name="joint_base" type="fixed">
-    <parent link="base_link"/>
-    <child link="link_0"/>
-  </joint>
-  <link name="link_0">
+  <link name="base">
     <visual>
       <geometry>
-        <!-- <mesh filename="package://fra333_lab1/meshes/link_0.stl"/> -->
         <mesh filename="package://robot_23_description/meshes/base.STL"/>
       </geometry>
@@ -27,5 +19,5 @@
   </link>
   <joint name="joint_1" type="revolute">
-    <parent link="link_0"/>
+    <parent link="base"/>
     <child link="link_1"/>
     <origin rpy="0 0 0" xyz="0 0 0.3"/>
@@ -44,5 +36,5 @@
     <parent link="link_1"/>
     <child link="link_2"/>
-    <origin rpy="1.57 0 0" xyz="0.16 0 0"/>
+    <origin rpy="1.57079632679 0 0" xyz="0.16 0 0"/>
     <axis xyz="0 0 1"/>
     <limit lower="-3.14" upper="3.14" effort="0.5" velocity="0.5"/>
@@ -83,18 +75,3 @@
     </visual>
   </link>
-  <!-- <joint name="joint_eff" type="fixed">
-    <parent link="link_3"/>
-    <child link="end_effector"/>
-    <origin rpy="1.57 0 1.57" xyz="0.35 0 0"/>
-    <axis xyz="0 0 1"/>
-  </joint>
-  <link name="end_effector">
-    <visual>
-      <origin rpy="0 0 0" xyz="0 0 0"/>
-      <geometry>
-        <mesh filename="package://robot_23_description/meshes/gripper.STL"/>
-      </geometry>
-      <material name="Orange"/>
-    </visual>
-  </link> -->
 </robot>
